Commit message: First env stands -> shape rewards and train

File: objects/drone.urdf (robot description, URDF)
Before this commit: robot drone, 5 links, 4 joints
Joints:
- joint base_to_BL: origin xyz=-0.09 0.13 0 rpy=0 0 0 -> xyz=-0.16 0.13 0 rpy=0 0 0
- joint base_to_BR: origin xyz=-0.09 -0.13 0 rpy=0 0 0 -> xyz=-0.16 -0.13 0 rpy=0 0 0
